File: LimeKeyboard.kicad_sch (KiCad schematic)
At the start: 87 parts

Commit message: made sure things are all local to this project
Parts:
- JP1, JP2, JP3, JP4, JP5, JP6, JP7, JP8: renamed from JP?; symbol SofleKeyboard-rescue:Jumper_NO_Small-Device -> Jumper:Jumper_2_Open
- SW31: renamed from SW?; symbol SofleKeyboard-rescue:Rotary_Encoder_Switch-Device -> Device:Rotary_Encoder_Switch
- W1: renamed from W?; symbol SofleKeyboard-rescue:Jumper-Device -> Jumper:Jumper_2_Bridged
- gave numbers to parts that had none: 77
Connections:
- net DATA: now also W1.1 (A)
- net ENCA: now also SW31.A
- net ENCB: now also SW31.B
- net GND: now also J2.2, JP1.2 (B), JP8.2 (B), SW31.C
- net SCL: now also JP3.2 (B), JP6.2 (B)
- net SDA: now also JP4.2 (B), JP5.2 (B)
- net SW31A: now also SW31.S1
- net SW31B: now also SW31.S2
- net VCC: now also J2.1, JP2.2 (B), JP7.2 (B)
- net i2c_d: now also W1.2 (B)
- net at J3.1 (P1): now also JP4.1 (A), JP8.1 (A)
- net at J3.2 (P2): now also JP3.1 (A), JP7.1 (A)
- net at J3.3 (P3): now also JP2.1 (A), JP6.1 (A)
- net at J3.4 (P4): now also JP1.1 (A), JP5.1 (A)
